File: VCA.kicad_pcb (KiCad board)
At the start: 2 copper layers, 50 x 50 mm, 32 parts, among them J1 Conn_01x02_Socket, J2 Conn_01x02_Socket, J3 Conn_01x02_Socket, J4 Conn_01x03_Female, J5 Conn_01x03_Female, Q1 BC547, Q2 BC547, Q3 BC547, U1 TL072

Commit message: added mounting holes
Parts:
- renumbered CV_AMOUNT1 to CV_AMOUNT, GAIN1 to GAIN, LEVEL_TRIM1 to LEVEL_TRIM, OFFSET_TRIM1 to OFFSET_TRIM
Routing:
- net -12V: track 109.8 -> 109.1 mm
Other:
- outline, holes or cut-outs redrawn
Changed lines of the file:
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@@
     (property "ki_keywords" "resistor variable")
     (attr through_hole)
-    (fp_text reference "GAIN1" (at 14.4 -2.45 -180) (layer "F.SilkS")
+    (fp_text reference "GAIN" (at 14.4 -2.45 180) (layer "F.SilkS")
         (effects (font (size 1 1) (thickness 0.15)))
     )
@@
     (property "ki_keywords" "resistor variable")
     (attr through_hole)
-    (fp_text reference "OFFSET_TRIM1" (at -4.625 -1.387944 -180) (layer "F.SilkS")
+    (fp_text reference "OFFSET_TRIM" (at -4.625 -1.387944 180) (layer "F.SilkS")
         (effects (font (size 1 1) (thickness 0.15)))
     )
@@
     (property "ki_keywords" "connector")
     (attr through_hole)
-    (fp_text reference "J2" (at 0 -2.68) (layer "F.SilkS")
+    (fp_text reference "J2" (at 2.5 -1.93 90) (layer "F.SilkS")
         (effects (font (size 1 1) (thickness 0.15)))
     )
@@
     (property "ki_keywords" "connector")
     (attr through_hole)
-    (fp_text reference "J3" (at 0 -2.33) (layer "F.SilkS")
+    (fp_text reference "J3" (at -2.652944 -1.685 270) (layer "F.SilkS")
         (effects (font (size 1 1) (thickness 0.15)))
     )
@@
     (property "ki_keywords" "resistor variable")
     (attr through_hole)
-    (fp_text reference "LEVEL_TRIM1" (at -4.575 -3.687944 -180) (layer "F.SilkS")
+    (fp_text reference "LEVEL_TRIM" (at -4.575 -3.687944 180) (layer "F.SilkS")
         (effects (font (size 1 1) (thickness 0.15)))
     )
@@
     (property "ki_keywords" "resistor variable")
     (attr through_hole)
-    (fp_text reference "CV_AMOUNT1" (at 14.6 -2.4 -180) (layer "F.SilkS")
+    (fp_text reference "CV_AMOUNT" (at 14.28 -2.4 180) (layer "F.SilkS")
         (effects (font (size 1 1) (thickness 0.15)))
     )
@@
   (gr_line (start 112.992056 64.756252) (end 112.747056 64.97)
     (stroke (width 0.15) (type default)) (layer "F.SilkS"))
+  (gr_circle (center 138.5 71.5) (end 140 71.5)
+    (stroke (width 0.1) (type default)) (fill none) (layer "Edge.Cuts"))
+  (gr_circle (center 103.25 106) (end 104.75 106)
+    (stroke (width 0.1) (type default)) (fill none) (layer "Edge.Cuts"))
   (gr_line (start 100 105) (end 100 63)
     (stroke (width 0.1) (type default)) (layer "Edge.Cuts"))
   (gr_line (start 104 109) (end 146 109)
     (stroke (width 0.1) (type default)) (layer "Edge.Cuts"))
+  (gr_circle (center 111.5 71.5) (end 111.5 70)
+    (stroke (width 0.1) (type default)) (fill none) (layer "Edge.Cuts"))
+  (gr_circle (center 146.75 106) (end 148.25 106)
+    (stroke (width 0.1) (type default)) (fill none) (layer "Edge.Cuts"))
   (gr_arc (start 146 59) (mid 148.828427 60.171573) (end 150 63)
     (stroke (width 0.1) (type default)) (layer "Edge.Cuts"))
@@
   (segment (start 131.642056 64.475) (end 131.642056 63.915) (width 1) (layer "F.Cu") (net 3))
   (segment (start 131.642056 63.915) (end 132.317056 63.24) (width 1) (layer "F.Cu") (net 3))
+  (segment (start 115.597056 70.402944) (end 115.597056 69.92) (width 0.4) (layer "F.Cu") (net 3))
   (segment (start 131.642056 64.475) (end 130.407056 63.24) (width 1) (layer "F.Cu") (net 3))
   (segment (start 116.497056 91.02) (end 116.697056 91.02) (width 0.4) (layer "F.Cu") (net 3))
@@
   (segment (start 114.997056 91.02) (end 116.497056 91.02) (width 0.4) (layer "F.Cu") (net 3))
   (segment (start 132.327056 63.23) (end 132.317056 63.24) (width 1) (layer "F.Cu") (net 3))
-  (segment (start 111.397056 73.02) (end 111.397056 77.92) (width 0.4) (layer "F.Cu") (net 3))
+  (segment (start 111.397056 74.602944) (end 115.597056 70.402944) (width 0.4) (layer "F.Cu") (net 3))
   (segment (start 111.397056 86.439239) (end 111.397056 87.42) (width 0.4) (layer "F.Cu") (net 3))
   (segment (start 147.867056 69.323503) (end 147.867056 65.68) (width 1) (layer "F.Cu") (net 3))
+  (segment (start 111.397056 77.92) (end 111.397056 74.602944) (width 0.4) (layer "F.Cu") (net 3))
   (segment (start 133.897056 78.82) (end 138.370559 78.82) (width 1) (layer "F.Cu") (net 3))
   (segment (start 145.417056 63.23) (end 132.327056 63.23) (width 1) (layer "F.Cu") (net 3))
@@
   (segment (start 114.497056 63.24) (end 113.944556 63.24) (width 1) (layer "F.Cu") (net 3))
   (segment (start 115.697056 65.82) (end 115.697056 63.34) (width 1) (layer "F.Cu") (net 3))
-  (segment (start 115.597056 69.92) (end 114.497056 69.92) (width 0.4) (layer "F.Cu") (net 3))
   (segment (start 131.642056 65.575) (end 131.642056 64.475) (width 1) (layer "F.Cu") (net 3))
   (segment (start 113.944556 63.24) (end 113.727056 63.4575) (width 1) (layer "F.Cu") (net 3))
@@
   (segment (start 115.697056 63.34) (end 115.797056 63.24) (width 1) (layer "F.Cu") (net 3))
   (segment (start 147.867056 65.68) (end 145.417056 63.23) (width 1) (layer "F.Cu") (net 3))
-  (segment (start 114.497056 69.92) (end 111.397056 73.02) (width 0.4) (layer "F.Cu") (net 3))
   (via (at 115.697056 65.82) (size 0.8) (drill 0.4) (layers "F.Cu" "B.Cu") (net 3))
   (via (at 111.397056 79.62) (size 0.8) (drill 0.4) (layers "F.Cu" "B.Cu") (net 3))

Commit message: added more silkscreen
Other:
- board text added: "INPUT"
- board text added: "OUTPUT"
- board text added: "SIGNAL_IN"
- board text added: "YOU KILLED IT"
- board text added: "if you are looking at this side you might have fucked up"
- board text removed: "SIGNAL"
Changed lines of the file:
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@@
     (property "ki_keywords" "R res resistor")
     (attr smd)
-    (fp_text reference "R4" (at -6.7 0) (layer "F.SilkS")
+    (fp_text reference "R4" (at -6.647056 0.03) (layer "F.SilkS")
         (effects (font (size 1 1) (thickness 0.15)))
     )
@@
     (property "ki_keywords" "R res resistor")
     (attr smd)
-    (fp_text reference "R1" (at -4.7 0) (layer "F.SilkS")
+    (fp_text reference "R1" (at -4.772056 0.03 180) (layer "F.SilkS")
         (effects (font (size 1 1) (thickness 0.15)))
     )
@@
     (property "ki_keywords" "R res resistor")
     (attr smd)
-    (fp_text reference "R9" (at 9.652944 0.03) (layer "F.SilkS")
+    (fp_text reference "R9" (at 6.652944 0.005) (layer "F.SilkS")
         (effects (font (size 1 1) (thickness 0.15)))
     )
@@
     (property "ki_keywords" "R res resistor")
     (attr smd)
-    (fp_text reference "R10" (at 3.3 0) (layer "F.SilkS")
+    (fp_text reference "R10" (at 5.502944 -0.045) (layer "F.SilkS")
         (effects (font (size 1 1) (thickness 0.15)))
     )
@@
     )
   )
+  (gr_line (start 123.8 84.55) (end 124.25 84.1)
+    (stroke (width 0.15) (type default)) (layer "F.SilkS"))
   (gr_line (start 101 89) (end 101 97)
     (stroke (width 0.15) (type default)) (layer "F.SilkS"))
+  (gr_line (start 123.7 83.925) (end 124.275 84.6)
+    (stroke (width 0.15) (type default)) (layer "F.SilkS"))
   (gr_line (start 145.65 88.125) (end 143.95 88.125)
     (stroke (width 0.15) (type default)) (layer "F.SilkS"))
@@
   (gr_line (start 104.5 81.25) (end 104.75 87.75)
     (stroke (width 0.15) (type default)) (layer "F.SilkS"))
+  (gr_line (start 124.75 85.65) (end 124.55 85.475)
+    (stroke (width 0.15) (type default)) (layer "F.SilkS"))
   (gr_line (start 147.05 86.575) (end 142.85 86.375)
     (stroke (width 0.15) (type default)) (layer "F.SilkS"))
@@
   (gr_line (start 134.922056 66.57) (end 135.157056 66.796248)
     (stroke (width 0.15) (type default)) (layer "F.SilkS"))
+  (gr_line (start 123.75 85.85) (end 124.175 85.5)
+    (stroke (width 0.15) (type default)) (layer "F.SilkS"))
   (gr_line (start 135.157056 67.318752) (end 134.922056 67.51)
     (stroke (width 0.15) (type default)) (layer "F.SilkS"))
@@
   (gr_line (start 146.8 87.025) (end 142.35 86.775)
     (stroke (width 0.15) (type default)) (layer "F.SilkS"))
+  (gr_line (start 123.7 85.325) (end 124.25 85.975)
+    (stroke (width 0.15) (type default)) (layer "F.SilkS"))
   (gr_line (start 145.15 93.4) (end 144.9 93.2)
     (stroke (width 0.15) (type default)) (layer "F.SilkS"))
@@
   (gr_line (start 143.95 92.425) (end 146.05 92.1)
     (stroke (width 0.15) (type default)) (layer "F.SilkS"))
+  (gr_line (start 124.55 85.475) (end 124.55 84.8)
+    (stroke (width 0.15) (type default)) (layer "F.SilkS"))
   (gr_line (start 107.802056 64.045) (end 112.777056 64.04)
     (stroke (width 0.15) (type default)) (layer "F.SilkS"))
@@
   (gr_line (start 101 89) (end 112 89)
     (stroke (width 0.15) (type default)) (layer "F.SilkS"))
+  (gr_line (start 124.55 84.8) (end 124.85 84.675)
+    (stroke (width 0.15) (type default)) (layer "F.SilkS"))
   (gr_line (start 136.902056 66.57) (end 136.627056 66.796248)
     (stroke (width 0.15) (type default)) (layer "F.SilkS"))
@@
   (gr_line (start 150 63) (end 150 105)
     (stroke (width 0.1) (type default)) (layer "Edge.Cuts"))
+  (gr_line (start 100.975 92.9) (end 110.55 92.9)
+    (stroke (width 0.15) (type default)) (layer "User.2"))
   (gr_line (start 60 92) (end 85 92)
     (stroke (width 0.15) (type default)) (layer "User.2"))
+  (gr_line (start 100.95 84.85) (end 110.525 84.85)
+    (stroke (width 0.15) (type default)) (layer "User.2"))
   (gr_line (start 92.4 43.6) (end 93.1 43.6)
     (stroke (width 0.15) (type default)) (layer "User.2"))
   (gr_line (start 93.1 43.6) (end 93.1 51.3)
     (stroke (width 0.15) (type default)) (layer "User.2"))
+  (gr_text "if you are looking at\nthis side you might have\nfucked up" (at 143.5 96 -90) (layer "B.SilkS")
+    (effects (font (size 1 1) (thickness 0.15)) (justify left bottom mirror))
+  )
   (gr_text "https://github.com/sirlilpanda/VCA" (at 111.45 103.85 180) (layer "B.SilkS")
     (effects (font (size 3 1) (thickness 0.15)) (justify left bottom mirror))
@@
     (effects (font (size 1 1) (thickness 0.15)) (justify left bottom))
   )
+  (gr_text "OUTPUT" (at 142.5 104 90) (layer "F.SilkS")
+    (effects (font (size 1 1) (thickness 0.15)) (justify left bottom))
+  )
   (gr_text "GND\n" (at 138.117056 66.37) (layer "F.SilkS")
     (effects (font (size 1 1) (thickness 0.15)) (justify left bottom))
@@
     (effects (font (size 1 1) (thickness 0.15)) (justify left bottom))
   )
-  (gr_text "SIGNAL\n" (at 101.55 79.95 90) (layer "F.SilkS")
+  (gr_text "SIGNAL_IN\n" (at 101.55 79.95 90) (layer "F.SilkS")
+    (effects (font (size 1 1) (thickness 0.15)) (justify left bottom))
+  )
+  (gr_text "INPUT" (at 109 103.5 90) (layer "F.SilkS")
+    (effects (font (size 1 1) (thickness 0.15)) (justify left bottom))
+  )
+  (gr_text "INPUT" (at 108.5 79.5 90) (layer "F.SilkS")
     (effects (font (size 1 1) (thickness 0.15)) (justify left bottom))
   )
+  (gr_text "YOU \nKILLED IT" (at 126.475 88.75 90) (layer "F.SilkS")
+    (effects (font (size 1 0.7) (thickness 0.15)) (justify left bottom))
+  )
   (segment (start 115.197056 93.22) (end 109.497056 87.52) (width 0.4) (layer "F.Cu") (net 1))
