File: VCA.kicad_sch (KiCad schematic)
At the start: 31 parts, among them J1 Conn_01x02_Socket, J2 Conn_01x02_Socket, J3 Conn_01x02_Socket, J4 Conn_01x03_Female, J5 Conn_01x03_Female, Q1 BC547, Q2 BC547, Q3 BC547, U1 TL072

Commit message: fixed?
Other:
- note added: "GAIN1"
- note removed: "GAIN"
Changed lines of the file:
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@@
     (stroke (width 0) (type default))
   )
-  (text "GAIN\n" (at 44.45 114.3 0)
+  (text "GAIN1\n" (at 44.45 114.3 0)
     (effects (font (size 1.27 1.27)) (justify left bottom))
   )

Commit message: added test points to the schmatic
Parts:
- added TP2, TP3, TP4: TestPoint_Probe, symbol Connector:TestPoint_Probe
- renumbered LEVEL_TRIM1 to LEVEL1, OFFSET_TRIM1 to OFFSET1
Connections:
- net AMout: now also TP3.1
- net carrierSignal: now also TP4.1
- net at CV_AMOUNT1.2, R3.1: now also TP2.1
Changed lines of the file:
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@@
   (junction (at 259.08 24.13) (diameter 0) (color 0 0 0 0)
   )
+  (junction (at 46.99 129.54) (diameter 0) (color 0 0 0 0)
+  )
   (junction (at 121.92 121.92) (diameter 0) (color 0 0 0 0)
   )
@@
   (junction (at 162.56 60.96) (diameter 0) (color 0 0 0 0)
   )
+  (junction (at 44.45 77.47) (diameter 0) (color 0 0 0 0)
+  )
   (junction (at 60.96 119.38) (diameter 0) (color 0 0 0 0)
   )
@@
   (junction (at 231.14 97.79) (diameter 0) (color 0 0 0 0)
   )
+  (junction (at 198.12 58.42) (diameter 0) (color 0 0 0 0)
+  )
   (junction (at 129.54 60.96) (diameter 0) (color 0 0 0 0)
   )
@@
     (stroke (width 0) (type default))
   )
-  (wire (pts (xy 204.47 58.42) (xy 194.31 58.42))
+  (wire (pts (xy 204.47 58.42) (xy 198.12 58.42))
     (stroke (width 0) (type default))
   )
@@
     (stroke (width 0) (type default))
   )
+  (wire (pts (xy 44.45 77.47) (xy 49.53 77.47))
+    (stroke (width 0) (type default))
+  )
   (wire (pts (xy 259.08 22.86) (xy 259.08 24.13))
     (stroke (width 0) (type default))
@@
     (stroke (width 0) (type default))
   )
+  (wire (pts (xy 46.99 129.54) (xy 50.8 129.54))
+    (stroke (width 0) (type default))
+  )
   (polyline (pts (xy 104.14 25.4) (xy 104.14 39.37))
     (stroke (width 0) (type default))
@@
     (stroke (width 0) (type default))
   )
+  (wire (pts (xy 198.12 58.42) (xy 194.31 58.42))
+    (stroke (width 0) (type default))
+  )
   (wire (pts (xy 60.96 110.49) (xy 60.96 119.38))
     (stroke (width 0) (type default))
@@
     (stroke (width 0) (type default))
   )
-  (wire (pts (xy 45.72 129.54) (xy 50.8 129.54))
+  (wire (pts (xy 45.72 129.54) (xy 46.99 129.54))
     (stroke (width 0) (type default))
   )
@@
     (stroke (width 0) (type default))
   )
-  (wire (pts (xy 31.75 77.47) (xy 49.53 77.47))
+  (wire (pts (xy 31.75 77.47) (xy 44.45 77.47))
     (stroke (width 0) (type default))
   )
@@
     )
   )
+  (symbol (lib_id "Connector:TestPoint_Probe") (at 44.45 77.47 0) (unit 1)
+    (in_bom yes) (on_board yes) (dnp no) (fields_autoplaced)
+    (property "Reference" "TP4" (at 48.26 74.6125 0)
+      (effects (font (size 1.27 1.27)) (justify left))
+    )
+    (property "Value" "TestPoint_Probe" (at 48.26 77.1525 0)
+      (effects (font (size 1.27 1.27)) (justify left))
+    )
+    (property "Footprint" "" (at 49.53 77.47 0)
+      (effects (font (size 1.27 1.27)) hide)
+    )
+    (property "Datasheet" "~" (at 49.53 77.47 0)
+      (effects (font (size 1.27 1.27)) hide)
+    )
+    (pin "1")
+    (instances
+      (project "VCA"
+        (path "/7f56cec0-dc04-41c0-a8fa-3d51520e0228"
+          (reference "TP4") (unit 1)
+        )
+      )
+    )
+  )
   (symbol (lib_name "GND_1") (lib_id "power:GND") (at 218.44 85.09 0) (unit 1)
     (in_bom yes) (on_board yes) (dnp no) (fields_autoplaced)
@@
     )
   )
+  (symbol (lib_id "Connector:TestPoint_Probe") (at 46.99 129.54 0) (unit 1)
+    (in_bom yes) (on_board yes) (dnp no) (fields_autoplaced)
+    (property "Reference" "TP2" (at 50.8 126.6825 0)
+      (effects (font (size 1.27 1.27)) (justify left))
+    )
+    (property "Value" "TestPoint_Probe" (at 50.8 129.2225 0)
+      (effects (font (size 1.27 1.27)) (justify left))
+    )
+    (property "Footprint" "" (at 52.07 129.54 0)
+      (effects (font (size 1.27 1.27)) hide)
+    )
+    (property "Datasheet" "~" (at 52.07 129.54 0)
+      (effects (font (size 1.27 1.27)) hide)
+    )
+    (pin "1")
+    (instances
+      (project "VCA"
+        (path "/7f56cec0-dc04-41c0-a8fa-3d51520e0228"
+          (reference "TP2") (unit 1)
+        )
+      )
+    )
+  )
   (symbol (lib_id "Device:R_Potentiometer") (at 81.28 99.06 0) (unit 1)
     (in_bom yes) (on_board yes) (dnp no) (fields_autoplaced)
-    (property "Reference" "LEVEL_TRIM1" (at 78.74 97.79 0)
+    (property "Reference" "LEVEL1" (at 78.74 97.79 0)
       (effects (font (size 1.27 1.27)) (justify right))
     )
@@
       (project "VCA"
         (path "/7f56cec0-dc04-41c0-a8fa-3d51520e0228"
-          (reference "LEVEL_TRIM1") (unit 1)
+          (reference "LEVEL1") (unit 1)
         )
       )
@@
     )
   )
+  (symbol (lib_id "Connector:TestPoint_Probe") (at 198.12 58.42 0) (unit 1)
+    (in_bom yes) (on_board yes) (dnp no) (fields_autoplaced)
+    (property "Reference" "TP3" (at 201.93 55.5625 0)
+      (effects (font (size 1.27 1.27)) (justify left))
+    )
+    (property "Value" "TestPoint_Probe" (at 201.93 58.1025 0)
+      (effects (font (size 1.27 1.27)) (justify left))
+    )
+    (property "Footprint" "" (at 203.2 58.42 0)
+      (effects (font (size 1.27 1.27)) hide)
+    )
+    (property "Datasheet" "~" (at 203.2 58.42 0)
+      (effects (font (size 1.27 1.27)) hide)
+    )
+    (pin "1")
+    (instances
+      (project "VCA"
+        (path "/7f56cec0-dc04-41c0-a8fa-3d51520e0228"
+          (reference "TP3") (unit 1)
+        )
+      )
+    )
+  )
   (symbol (lib_id "power:GND") (at 252.73 40.64 270) (unit 1)
     (in_bom yes) (on_board yes) (dnp no)
@@
   (symbol (lib_id "Device:R_Potentiometer") (at 120.65 40.64 90) (unit 1)
     (in_bom yes) (on_board yes) (dnp no)
-    (property "Reference" "OFFSET_TRIM1" (at 120.65 45.72 90)
+    (property "Reference" "OFFSET1" (at 120.65 45.72 90)
       (effects (font (size 1.27 1.27)))
     )
@@
       (project "VCA"
         (path "/7f56cec0-dc04-41c0-a8fa-3d51520e0228"
-          (reference "OFFSET_TRIM1") (unit 1)
-        )
-      )
+          (reference "OFFSET1") (unit 1)
+        )
+      )

Commit message: updated gbrs
Parts:
- removed TP2, TP3, TP4: TestPoint_Probe, symbol Connector:TestPoint_Probe
Changed lines of the file:
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@@
   (junction (at 259.08 24.13) (diameter 0) (color 0 0 0 0)
   )
-  (junction (at 46.99 129.54) (diameter 0) (color 0 0 0 0)
-  )
   (junction (at 121.92 121.92) (diameter 0) (color 0 0 0 0)
   )
@@
   (junction (at 162.56 60.96) (diameter 0) (color 0 0 0 0)
   )
-  (junction (at 44.45 77.47) (diameter 0) (color 0 0 0 0)
-  )
   (junction (at 60.96 119.38) (diameter 0) (color 0 0 0 0)
   )
@@
   (junction (at 231.14 97.79) (diameter 0) (color 0 0 0 0)
   )
-  (junction (at 198.12 58.42) (diameter 0) (color 0 0 0 0)
-  )
   (junction (at 129.54 60.96) (diameter 0) (color 0 0 0 0)
   )
@@
     (stroke (width 0) (type default))
   )
-  (wire (pts (xy 204.47 58.42) (xy 198.12 58.42))
-    (stroke (width 0) (type default))
-  )
   (wire (pts (xy 110.49 102.87) (xy 106.68 102.87))
     (stroke (width 0) (type default))
@@
     (stroke (width 0) (type default))
   )
-  (wire (pts (xy 44.45 77.47) (xy 49.53 77.47))
+  (wire (pts (xy 31.75 77.47) (xy 49.53 77.47))
     (stroke (width 0) (type default))
   )
@@
     (stroke (width 0) (type default))
   )
-  (wire (pts (xy 46.99 129.54) (xy 50.8 129.54))
+  (wire (pts (xy 45.72 129.54) (xy 50.8 129.54))
     (stroke (width 0) (type default))
   )
@@
     (stroke (width 0) (type default))
   )
-  (wire (pts (xy 198.12 58.42) (xy 194.31 58.42))
+  (wire (pts (xy 194.31 58.42) (xy 204.47 58.42))
     (stroke (width 0) (type default))
   )
@@
     (stroke (width 0) (type default))
   )
-  (wire (pts (xy 45.72 129.54) (xy 46.99 129.54))
-    (stroke (width 0) (type default))
-  )
   (wire (pts (xy 218.44 77.47) (xy 218.44 76.2))
     (stroke (width 0) (type default))
@@
   )
   (polyline (pts (xy 200.66 139.7) (xy 38.1 139.7))
-    (stroke (width 0) (type default))
-  )
-  (wire (pts (xy 31.75 77.47) (xy 44.45 77.47))
     (stroke (width 0) (type default))
   )
@@
     )
   )
-  (symbol (lib_id "Connector:TestPoint_Probe") (at 44.45 77.47 0) (unit 1)
-    (in_bom yes) (on_board yes) (dnp no) (fields_autoplaced)
-    (property "Reference" "TP4" (at 48.26 74.6125 0)
-      (effects (font (size 1.27 1.27)) (justify left))
-    )
-    (property "Value" "TestPoint_Probe" (at 48.26 77.1525 0)
-      (effects (font (size 1.27 1.27)) (justify left))
-    )
-    (property "Footprint" "" (at 49.53 77.47 0)
-      (effects (font (size 1.27 1.27)) hide)
-    )
-    (property "Datasheet" "~" (at 49.53 77.47 0)
-      (effects (font (size 1.27 1.27)) hide)
-    )
-    (pin "1")
-    (instances
-      (project "VCA"
-        (path "/7f56cec0-dc04-41c0-a8fa-3d51520e0228"
-          (reference "TP4") (unit 1)
-        )
-      )
-    )
-  )
   (symbol (lib_name "GND_1") (lib_id "power:GND") (at 218.44 85.09 0) (unit 1)
     (in_bom yes) (on_board yes) (dnp no) (fields_autoplaced)
@@
         (path "/97e53a6b-0ed5-4440-b325-ee853eede691/883082d7-29db-4207-b92d-03cb522cabba"
           (reference "R7") (unit 1)
-        )
-      )
-    )
-  )
-  (symbol (lib_id "Connector:TestPoint_Probe") (at 46.99 129.54 0) (unit 1)
-    (in_bom yes) (on_board yes) (dnp no) (fields_autoplaced)
-    (property "Reference" "TP2" (at 50.8 126.6825 0)
-      (effects (font (size 1.27 1.27)) (justify left))
-    )
-    (property "Value" "TestPoint_Probe" (at 50.8 129.2225 0)
-      (effects (font (size 1.27 1.27)) (justify left))
-    )
-    (property "Footprint" "" (at 52.07 129.54 0)
-      (effects (font (size 1.27 1.27)) hide)
-    )
-    (property "Datasheet" "~" (at 52.07 129.54 0)
-      (effects (font (size 1.27 1.27)) hide)
-    )
-    (pin "1")
-    (instances
-      (project "VCA"
-        (path "/7f56cec0-dc04-41c0-a8fa-3d51520e0228"
-          (reference "TP2") (unit 1)
         )
       )
@@
         )
       )
-    )
-  )
-  (symbol (lib_id "Connector:TestPoint_Probe") (at 198.12 58.42 0) (unit 1)
-    (in_bom yes) (on_board yes) (dnp no) (fields_autoplaced)
-    (property "Reference" "TP3" (at 201.93 55.5625 0)
-      (effects (font (size 1.27 1.27)) (justify left))
-    )
-    (property "Value" "TestPoint_Probe" (at 201.93 58.1025 0)
-      (effects (font (size 1.27 1.27)) (justify left))
-    )
-    (property "Footprint" "" (at 203.2 58.42 0)
-      (effects (font (size 1.27 1.27)) hide)
-    )
-    (property "Datasheet" "~" (at 203.2 58.42 0)
-      (effects (font (size 1.27 1.27)) hide)
-    )
-    (pin "1")
-    (instances
-      (project "VCA"
-        (path "/7f56cec0-dc04-41c0-a8fa-3d51520e0228"
-          (reference "TP3") (unit 1)
-        )
-      )
